File: pcb/Hackpad.kicad_sch (KiCad schematic)
At the start: 26 parts, among them J1 Conn_01x04_Pin, SW1 SW_Push_45deg, SW10 RotaryEncoder_Switch, SW2 SW_Push_45deg, SW3 SW_Push_45deg, SW4 SW_Push_45deg, SW5 SW_Push_45deg, SW6 SW_Push_45deg, SW7 SW_Push_45deg, SW8 SW_Push_45deg, SW9 SW_Push_45deg, U1 MOUDLE-SEEEDUINO-XIAO

Commit message: Add files via upload
Parts:
- D10, D11, D12, D13: footprint footprints.pretty:SK6812MINI-E_fixed -> LED_SMD:LED_SK6812MINI-E_3.2x2.8mm_P1.5mm_ReverseMount
Connections:
- net BTN: now also D14.1 (K); no longer D14.2 (A)
- net Row 0: now also D14.2 (A); no longer D14.1 (K)
Other:
- moved on the sheet: D14
Changed lines of the file:
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@@
 	(wire
 		(pts
-			(xy 170.18 101.6) (xy 186.69 101.6)
+			(xy 217.17 81.28) (xy 226.06 81.28)
 		)
 		(stroke
@@
 	(wire
 		(pts
-			(xy 217.17 81.28) (xy 226.06 81.28)
+			(xy 170.18 101.6) (xy 186.69 101.6)
 		)
 		(stroke
@@
 			)
 		)
-		(property "Footprint" "footprints.pretty:SK6812MINI-E_fixed"
+		(property "Footprint" "LED_SMD:LED_SK6812MINI-E_3.2x2.8mm_P1.5mm_ReverseMount"
 			(at 182.88 146.05 0)
 			(hide yes)
@@
 			)
 		)
-		(property "Footprint" "footprints.pretty:SK6812MINI-E_fixed"
+		(property "Footprint" "LED_SMD:LED_SK6812MINI-E_3.2x2.8mm_P1.5mm_ReverseMount"
 			(at 236.22 146.05 0)
 			(hide yes)
@@
 	(symbol
 		(lib_id "Diode:1N914")
-		(at 217.17 77.47 90)
+		(at 217.17 77.47 270)
 		(unit 1)
 		(body_style 1)
@@
 					(size 1.27 1.27)
 				)
-				(justify right)
+				(justify left)
 			)
 		)
@@
 					(size 1.27 1.27)
 				)
-				(justify right)
+				(justify left)
 			)
 		)
 		(property "Footprint" "Diode_THT:D_DO-35_SOD27_P7.62mm_Horizontal"
-			(at 221.615 77.47 0)
+			(at 212.725 77.47 0)
 			(hide yes)
 			(show_name no)
@@
 			)
 		)
-		(property "Footprint" "footprints.pretty:SK6812MINI-E_fixed"
+		(property "Footprint" "LED_SMD:LED_SK6812MINI-E_3.2x2.8mm_P1.5mm_ReverseMount"
 			(at 209.55 146.05 0)
 			(hide yes)
@@
 			)
 		)
-		(property "Footprint" "footprints.pretty:SK6812MINI-E_fixed"
+		(property "Footprint" "LED_SMD:LED_SK6812MINI-E_3.2x2.8mm_P1.5mm_ReverseMount"
 			(at 156.21 146.05 0)
 			(hide yes)
